File: kicad/IO.kicad_sch (KiCad schematic)
At the start: 12 parts, among them SW1 1571407-1, U17 NC7WZ16

Commit message: kicad updated
Changed lines of the file:
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@@
 (kicad_sch
-	(version 20250114)
+	(version 20231120)
 	(generator "eeschema")
-	(generator_version "9.0")
+	(generator_version "8.0")
 	(paper "A4")
 	(junction
