File: kicad/Stabilizers.kicad_sch (KiCad schematic)
At the start: 92 parts, among them J1 MSTBA2.5/2-G-5.08 1757242, P1 PAD, P10 +12VA, P11 -15V_CN, P12 -15V_CP, P13 -12VA, P14 -1VA, P2 +12V, P3 +5VA, P4 +3V3A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

Commit message: kicad updated
Parts:
- U7, U8, U9: footprint Package_DFN_QFN:DFN-12-1EP_3x3mm_P0.5mm_EP1.6x2.5mm_ThermalVias -> Package_DFN_QFN:DFN-12-1EP_2x3mm_P0.45mm_EP0.64x2.4mm
Changed lines of the file:
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@@
 (kicad_sch
-	(version 20250114)
+	(version 20231120)
 	(generator "eeschema")
-	(generator_version "9.0")
+	(generator_version "8.0")
 	(paper "A4")
 	(junction
@@
 			)
 		)
-		(property "Footprint" "Package_DFN_QFN:DFN-12-1EP_3x3mm_P0.5mm_EP1.6x2.5mm_ThermalVias"
+		(property "Footprint" "Package_DFN_QFN:DFN-12-1EP_2x3mm_P0.45mm_EP0.64x2.4mm"
 			(at 139.7 193.04 0)
 			(effects
@@
 			)
 		)
-		(property "Comm" ""
-			(at 139.7 193.04 0)
-			(effects
-				(font
-					(size 1.27 1.27)
-				)
-			)
-		)
-		(property "Vendor" ""
-			(at 139.7 193.04 0)
-			(effects
-				(font
-					(size 1.27 1.27)
-				)
-				(hide yes)
-			)
-		)
 		(pin "11"
 		)
@@
 			)
 		)
-		(property "Footprint" "Package_DFN_QFN:DFN-12-1EP_3x3mm_P0.5mm_EP1.6x2.5mm_ThermalVias"
+		(property "Footprint" "Package_DFN_QFN:DFN-12-1EP_2x3mm_P0.45mm_EP0.64x2.4mm"
 			(at 139.7 123.19 0)
 			(effects
@@
 			)
 		)
-		(property "Comm" ""
-			(at 139.7 123.19 0)
-			(effects
-				(font
-					(size 1.27 1.27)
-				)
-			)
-		)
-		(property "Vendor" ""
-			(at 139.7 123.19 0)
-			(effects
-				(font
-					(size 1.27 1.27)
-				)
-				(hide yes)
-			)
-		)
 		(pin "10"
 		)
@@
 			)
 		)
-		(property "Footprint" "Package_DFN_QFN:DFN-12-1EP_3x3mm_P0.5mm_EP1.6x2.5mm_ThermalVias"
+		(property "Footprint" "Package_DFN_QFN:DFN-12-1EP_2x3mm_P0.45mm_EP0.64x2.4mm"
 			(at 139.7 165.1 0)
 			(effects
@@
 			(at 139.7 165.1 0)
 			(effects
-				(font
-					(size 1.27 1.27)
-				)
-				(hide yes)
-			)
-		)
-		(property "Comm" ""
-			(at 139.7 165.1 0)
-			(effects
-				(font
-					(size 1.27 1.27)
-				)
-			)
-		)
-		(property "Vendor" ""
-			(at 139.7 165.1 0)
-			(effects
